Commit message: update model and task config files for boltnut, exploration, and balll sorting tasks

File: assets/industreal/urdf/ball_class_base.urdf (robot description, URDF)
Before this commit: robot classification_ball, 1 links, 0 joints
Links:
- link ball: geometry collision mesh filename=../mesh/TVB_mesh/ball_task_base_square.obj scale=0.35 1.2 1; visual mesh filename=../mesh/TVB_mesh/ball_task_base_square.obj scale=0.35 1.2 1

File: assets/industreal/urdf/ball_class_golf.urdf (robot description, URDF)
Before this commit: robot classification_ball, 1 links, 0 joints
Links:
- removed link ball
- added link golf_ball; collision mesh filename=../mesh/TVB_mesh/ball_task_golf.obj; visual mesh filename=../mesh/TVB_mesh/ball_task_golf.obj

File: assets/industreal/urdf/ball_class_tabletennis.urdf (robot description, URDF)
Before this commit: robot classification_ball, 1 links, 0 joints
Links:
- removed link ball
- added link pingpong_ball; collision mesh filename=../mesh/TVB_mesh/sphere.obj; visual mesh filename=../mesh/TVB_mesh/sphere.obj
