Commit message: update gears urdf for gear assembly task

File: assets/industreal/urdf/industreal_gear_base.urdf (robot description, URDF)
Before this commit: robot industreal_gear_base, 1 links, 0 joints
Links:
- link industreal_gear_base: geometry collision mesh filename=../mesh/TVB_mesh/gear_base_origin_Mar21.obj scale=2 2 2; visual mesh filename=../mesh/TVB_mesh/gear_base_origin_Mar21.obj scale=2 2 2

File: assets/industreal/urdf/industreal_gear_large.urdf (robot description, URDF)
Before this commit: robot industreal_gear_large, 1 links, 0 joints
Links:
- link industreal_gear_large: geometry collision mesh filename=../mesh/TVB_mesh/gear_large_origin_Mar21.obj scale=2 2 2; visual mesh filename=../mesh/TVB_mesh/gear_large_origin_Mar21.obj scale=2 2 2

File: assets/industreal/urdf/industreal_gear_medium.urdf (robot description, URDF)
Before this commit: robot industreal_gear_medium, 1 links, 0 joints
Links:
- link industreal_gear_medium: geometry collision mesh filename=../mesh/TVB_mesh/gear_medium_origin_update_Mar21.obj scale=1.95 1.95 1.95; visual mesh filename=../mesh/TVB_mesh/gear_medium_origin_update_Mar21.obj scale=1.95 1.95 1.95

File: assets/industreal/urdf/industreal_gear_small.urdf (robot description, URDF)
Before this commit: robot industreal_gear_small, 1 links, 0 joints
Links:
- link industreal_gear_small: geometry collision mesh filename=../mesh/TVB_mesh/gear_small_origin_Mar21.obj scale=2 2 2; visual mesh filename=../mesh/TVB_mesh/gear_small_origin_Mar21.obj scale=2 2 2

Commit message: update resources and codebase for rl gear assembly

File: assets/industreal/urdf/industreal_gear_base.urdf (robot description, URDF)
Before this commit: robot industreal_gear_base, 1 links, 0 joints
Links:
- link industreal_gear_base: geometry collision mesh filename=../mesh/TVB_mesh/manifeel_gear_base.obj scale=1 1 1; visual mesh filename=../mesh/TVB_mesh/manifeel_gear_base.obj scale=1 1 1

File: assets/industreal/urdf/industreal_gear_large.urdf (robot description, URDF)
Before this commit: robot industreal_gear_large, 1 links, 0 joints
Links:
- link industreal_gear_large: geometry collision mesh filename=../mesh/TVB_mesh/manifeel_gear_large.obj scale=1 1 1; visual mesh filename=../mesh/TVB_mesh/manifeel_gear_large.obj scale=1 1 1

File: assets/industreal/urdf/industreal_gear_medium.urdf (robot description, URDF)
Before this commit: robot industreal_gear_medium, 1 links, 0 joints
Links:
- link industreal_gear_medium: geometry collision mesh filename=../mesh/TVB_mesh/manifeel_gear_medium.obj scale=0.96 0.96 0.96; visual mesh filename=../mesh/TVB_mesh/manifeel_gear_medium.obj scale=0.96 0.96 0.96

File: assets/industreal/urdf/industreal_gear_small.urdf (robot description, URDF)
Before this commit: robot industreal_gear_small, 1 links, 0 joints
Links:
- link industreal_gear_small: geometry collision mesh filename=../mesh/TVB_mesh/manifeel_gear_small.obj scale=1 1 1; visual mesh filename=../mesh/TVB_mesh/manifeel_gear_small.obj scale=1 1 1
