Commit message: update assests for usb/power plug insertion task

File: assets/industreal/urdf/USB_plug.urdf (robot description, URDF)
Before this commit: robot USB_plug, 1 links, 0 joints
Links:
- link USB_plug: geometry collision mesh filename=../mesh/TVB_mesh/manifeel_usb_plug.obj; visual mesh filename=../mesh/TVB_mesh/manifeel_usb_plug.obj

File: assets/industreal/urdf/USB_socket.urdf (robot description, URDF)
Before this commit: robot USB_socket, 1 links, 0 joints
Links:
- link USB_socket: geometry collision mesh filename=../mesh/TVB_mesh/manifeel_usb_socket.obj; visual mesh filename=../mesh/TVB_mesh/manifeel_usb_socket.obj

File: assets/industreal/urdf/power_plug.urdf (robot description, URDF)
Before this commit: robot power_plug_medium, 1 links, 0 joints
Links:
- removed link power_plug_medium
- added link power_plug; collision mesh filename=../mesh/TVB_mesh/manifeel_power_plug.obj; visual mesh filename=../mesh/TVB_mesh/manifeel_power_plug.obj

File: assets/industreal/urdf/power_socket.urdf (robot description, URDF)
Before this commit: robot power_socekt_medium, 1 links, 0 joints
Links:
- removed link power_socekt_medium
- added link power_socket; collision mesh filename=../mesh/TVB_mesh/manifeel_power_socket.obj; visual mesh filename=../mesh/TVB_mesh/manifeel_power_socket.obj
