Commit message: update task gear class for in-hand randomization and gear urdf for color change and a bigger scaled shape

File: assets/industreal/urdf/industreal_gear_medium.urdf (robot description, URDF)
Before this commit: robot industreal_gear_medium, 1 links, 0 joints
Links:
- link industreal_gear_medium: geometry collision mesh filename=../mesh/TVB_mesh/gear_medium_origin_update_Mar21.obj scale=1.96 1.96 1.96; visual mesh filename=../mesh/TVB_mesh/gear_medium_origin_update_Mar21.obj scale=1.96 1.96 1.96

Commit message: update resource and code for rl gear assembly

File: assets/industreal/urdf/industreal_gear_medium.urdf (robot description, URDF)
Before this commit: robot industreal_gear_medium, 1 links, 0 joints
Links:
- link industreal_gear_medium: geometry collision mesh filename=../mesh/TVB_mesh/manifeel_gear_medium.obj scale=1.0 1.0 1.0; visual mesh filename=../mesh/TVB_mesh/manifeel_gear_medium.obj scale=1.0 1.0 1.0

Commit message: udpate medium gear size (urdf) for gear assembly task

File: assets/industreal/urdf/industreal_gear_medium.urdf (robot description, URDF)
Before this commit: robot industreal_gear_medium, 1 links, 0 joints
Links:
- link industreal_gear_medium: geometry collision mesh filename=../mesh/TVB_mesh/manifeel_gear_medium.obj scale=0.98 0.98 0.98; visual mesh filename=../mesh/TVB_mesh/manifeel_gear_medium.obj scale=0.98 0.98 0.98

Commit message: update gear task assets

File: assets/industreal/urdf/industreal_gear_medium.urdf (robot description, URDF)
Before this commit: robot industreal_gear_medium, 1 links, 0 joints
Links:
- link industreal_gear_medium: geometry collision mesh filename=../mesh/TVB_mesh/manifeel_gear_medium.obj scale=0.965 0.965 0.965; visual mesh filename=../mesh/TVB_mesh/manifeel_gear_medium.obj scale=0.965 0.965 0.965
